Commit message: working version

File: ebs_description/urdf/ebs_tractor.urdf (robot description, URDF)
Before this commit: robot ebs_tractor, 6 links, 5 joints
Joints:
- joint hokuyo_joint: origin (none) -> xyz=0 0 0.67 rpy=0 0 1.570796326

Commit message: working simulation

File: ebs_description/urdf/ebs_tractor.urdf (robot description, URDF)
Before this commit: robot ebs_tractor, 6 links, 5 joints
Joints:
- joint steering_joint: limit lower=-0.523599 upper=0.523599 effort=1000.0 velocity=10 -> lower=-0.95993 upper=0.95993 effort=1000.0 velocity=10
